File: LuminchOne.brd (EAGLE design)
At the start: 12 parts, among them J1 POWER_JACKPTH, Q1 BC337, U1 TINY85-20-DIP

Commit message: EAGLE Files
Parts:
- moved JP3 1.27 mm to (3.81, 27.9)
Routing:
- net VCC: track 39.7 -> 38.2 mm
- net V0: track 12.0 -> 12.5 mm
Changed lines of the file:
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@@
 <element name="Q1" library="transistor-npn-biggerHoles" package="TO92" value="BC337" x="3.81" y="38.1" rot="R270"/>
 <element name="JP2" library="SparkFun-Connectors" package="1X02" value="M02PTH" x="6.35" y="33.02" rot="R180"/>
-<element name="JP3" library="SparkFun-Connectors" package="1X03" value="VCC" x="3.81" y="29.21" rot="R270"/>
+<element name="JP3" library="SparkFun-Connectors" package="1X03" value="VCC" x="3.81" y="27.94" rot="R270"/>
 <element name="R1" library="SparkFun-Resistors" package="AXIAL-0.4" value="220" x="12.7" y="39.37" rot="R180"/>
 <element name="R2" library="SparkFun-Resistors" package="AXIAL-0.6" value="18" x="11.43" y="43.18" rot="R180"/>
@@
 <wire x1="5.08" y1="8.89" x2="3.81" y2="12.7" width="0.6096" layer="16"/>
 <wire x1="3.81" y1="12.7" x2="3.81" y2="17.78" width="0.6096" layer="16"/>
-<wire x1="3.81" y1="29.21" x2="8.89" y2="29.21" width="0.6096" layer="16"/>
-<wire x1="3.81" y1="29.21" x2="2.54" y2="29.21" width="0.6096" layer="16"/>
-<wire x1="2.54" y1="29.21" x2="1.27" y2="27.94" width="0.6096" layer="16"/>
-<wire x1="1.27" y1="27.94" x2="1.27" y2="19.05" width="0.6096" layer="16"/>
-<wire x1="1.27" y1="19.05" x2="2.54" y2="17.78" width="0.6096" layer="16"/>
-<wire x1="2.54" y1="17.78" x2="3.81" y2="17.78" width="0.6096" layer="16"/>
 <wire x1="8.89" y1="29.21" x2="8.89" y2="31.75" width="0.6096" layer="16"/>
 <wire x1="8.89" y1="31.75" x2="7.62" y2="33.02" width="0.6096" layer="16"/>
@@
 <wire x1="12.7" y1="34.29" x2="11.43" y2="34.29" width="0.6096" layer="16"/>
 <wire x1="11.43" y1="34.29" x2="8.89" y2="31.75" width="0.6096" layer="16"/>
+<wire x1="3.81" y1="17.78" x2="1.27" y2="20.32" width="0.6096" layer="16"/>
+<wire x1="1.27" y1="20.32" x2="1.27" y2="26.67" width="0.6096" layer="16"/>
+<wire x1="1.27" y1="26.67" x2="2.54" y2="27.94" width="0.6096" layer="16"/>
+<wire x1="2.54" y1="27.94" x2="3.81" y2="27.94" width="0.6096" layer="16"/>
+<wire x1="3.81" y1="27.94" x2="7.62" y2="27.94" width="0.6096" layer="16"/>
+<wire x1="7.62" y1="27.94" x2="8.89" y2="29.21" width="0.6096" layer="16"/>
 </signal>
 <signal name="GND">
@@
 <contactref element="U1" pad="3"/>
 <contactref element="JP3" pad="3"/>
-<wire x1="3.81" y1="24.13" x2="12.7" y2="24.13" width="0.6096" layer="16"/>
+<wire x1="3.81" y1="22.86" x2="6.35" y2="22.86" width="0.6096" layer="16"/>
+<wire x1="6.35" y1="22.86" x2="7.62" y2="24.13" width="0.6096" layer="16"/>
+<wire x1="7.62" y1="24.13" x2="12.7" y2="24.13" width="0.6096" layer="16"/>
 <wire x1="12.7" y1="24.13" x2="13.97" y2="22.86" width="0.6096" layer="16"/>
 <wire x1="13.97" y1="22.86" x2="13.97" y2="21.59" width="0.6096" layer="16"/>
